File: walleEagle/Wall-E/motor_connector_board.sch (EAGLE design)
At the start: 32 parts, among them U1 JST_SH_4, U2 JST_SH_6, U3 JST_SH_6, U4 MOLEX_ULTRAFIT, U5 SMC

Commit message: completely redid routing and made standoffs symmetrical
Other:
- note added: "0.2"
- note removed: "0.1"
Changed lines of the file:
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@@
 <?xml version="1.0" encoding="utf-8"?>
 <!DOCTYPE eagle SYSTEM "eagle.dtd">
-<eagle version="8.5.0">
+<eagle version="8.5.2">
 <drawing>
 <settings>
@@
 <plain>
 <text x="350.52" y="7.62" size="5.08" layer="94">Dexter Watkins</text>
-<text x="421.64" y="7.62" size="3.81" layer="94">0.1</text>
+<text x="421.64" y="7.62" size="3.81" layer="94">0.2</text>
 <text x="2.54" y="269.24" size="6.4516" layer="91">Wall-E</text>
 <text x="2.54" y="261.62" size="3.81" layer="91">Motor Connnection Board</text>
